Commit message: most recent -jash ke saath vala

File: hybrid_a_star_ws/src/Hybrid_A_Star/model/car_model/default.urdf (robot description, URDF)
Before this commit: robot car, 1 links, 0 joints
Links:
- link ground_link: geometry visual mesh filename=package://hybrid_a_star/model/car_model/CAR_original.dae scale=11 11 11

Commit message: working ttok smaller map 20Hz avoids obstacles does everything

File: hybrid_a_star_ws/src/Hybrid_A_Star/model/car_model/default.urdf (robot description, URDF)
Before this commit: robot car, 1 links, 0 joints
Links:
- link ground_link: geometry visual mesh filename=package://hybrid_a_star/model/car_model/CAR_original.dae scale=1.1 1.1 1.1
